File: led-driver.kicad_pcb (KiCad board)
At the start: 2 copper layers, 34.3 x 31.7 mm, 23 parts, among them J1 48VDC IN, J2 ENABLE, J3 ADJ, J4 LED, Q1 ZXMP7A17KTC, U1 LM3409HV

Commit message: Rescue symbols, minor revisions to PCB
This commits previous work that took place sporadically between the last
commit a year and a half ago, and now.
Parts:
- R1: moved to B.Cu
- moved R1 5.89 mm to (165.8, 120.0), turned to 0 degrees
- moved REF*** 1.56 mm to (164.6, 105.2)
- moved L1 0.23 mm to (163.6, 114.3)
Routing:
- net GND: track 1.90 -> 9.42 mm, vias 0 -> 10
- net Net-(C5-Pad1): track 21.9 -> 18.5 mm, vias 0 -> 1
- net Net-(C2-Pad1): track 6.73 -> 7.81 mm, vias 1 -> 0
Other:
- board text added: "Const. Current LED Driver Ver 1 (May 2019) David Phillips https://nah.nz/"
- board text removed: "Const. Current LED Driver Rev 1 David Phillips https://sighup.nz/"

Commit message: Reduce clearances, margin on MSOP footprint
Reduction of the soldermask margin allows soldermask to be placed between the
landing pads for the leads, which should aid soldering. Reduction of the
pad clearance should stop DRC from complaining about nets too close together.
Other:
- board text added: "Const. Current LED Driver Ver 1.1 (May 2019) David Phillips https://nah.nz/"
- board text removed: "Const. Current LED Driver Ver 1 (May 2019) David Phillips https://nah.nz/"
Changed lines of the file:
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@@
     (descr "MSE Package; 10-Lead Plastic MSOP, Exposed Die Pad (see Linear Technology 05081664_I_MSE.pdf)")
     (tags "SSOP 0.5")
+    (solder_mask_margin 0.04)
+    (clearance 0.09)
     (attr smd)
     (fp_text reference U1 (at 0 3.048 180) (layer B.SilkS)
@@
     (effects (font (size 1 1) (thickness 0.2)) (justify left mirror))
   )
-  (gr_text "Const. Current LED Driver\nVer 1 (May 2019)\nDavid Phillips\nhttps://nah.nz/" (at 179.07 101.6) (layer B.SilkS)
+  (gr_text "Const. Current LED Driver\nVer 1.1 (May 2019)\nDavid Phillips\nhttps://nah.nz/" (at 179.07 101.6) (layer B.SilkS)
     (effects (font (size 0.7 0.7) (thickness 0.15)) (justify left mirror))
   )

Commit message: Increase UVLO turn-on to 43 V
The initial design assumed that the UVLO was a feature of the LM3409 not needed
by this board. It was set at the datasheet values of 10.1 V turn-on with 1.1 V
of hysteresis. However, during testing, I have found that the supply will sink
a maximum of around 600 mA into the load when operated into dropout. The LM3409
datasheet confirms that this is expected behaviour. Since the supply is
designed for LEDs modules with a forward voltage of 37 V, this patch changes
the UVLO to just over 43 volts, meaning that we do not run the LEDs above the
supply's design current of 450 mA.
Parts:
- R2: value 6.98kΩ -> 1.47kΩ
Changed lines of the file:
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@@
       (effects (font (size 1 1) (thickness 0.15)))
     )
-    (fp_text value 6.98kΩ (at 0 1.75 270) (layer F.Fab)
+    (fp_text value 1.47kΩ (at 0 1.75 270) (layer F.Fab)
       (effects (font (size 1 1) (thickness 0.15)))
     )
