File: led-driver.sch (KiCad schematic (older format))
At the start: 18 parts, among them J1 48VDC IN, J2 ENABLE, J3 ADJ, J4 LED, Q1 ZXMP7A17KTC, U1 LM3409HV

Commit message: Fix up symbols
Parts:
- C1, C2, C3, C4, C5: symbol led-driver-rescue:C_Small -> Device:C_Small
- D1: symbol led-driver-rescue:D_Schottky_Small_ALT -> Device:D_Schottky_Small_ALT
- J1, J3, J4: symbol led-driver-rescue:CONN_01X02 -> Connector_Generic:Conn_01x02
- J2: symbol led-driver-rescue:CONN_01X03 -> Connector_Generic:Conn_01x03
- L1: symbol led-driver-rescue:L_Small -> Device:L_Small
- Q1: symbol led-driver-rescue:Q_PMOS_GDS -> Device:Q_PMOS_GDS
- R1, R2, R3, R4, R5: symbol led-driver-rescue:R_Small -> Device:R_Small
- U1: symbol led-driver-rescue:LM3409-RESCUE-led-driver-new -> led-driver:LM3409
Changed lines of the file:
@@
 $EndDescr
 $Comp
-L led-driver-rescue:R_Small R4
+L Device:R_Small R4
 U 1 1 59AE9865
 P 5800 3300
@@
 $EndComp
 $Comp
-L led-driver-rescue:D_Schottky_Small_ALT D1
+L Device:D_Schottky_Small_ALT D1
 U 1 1 59AE99D5
 P 5800 4000
@@
 $EndComp
 $Comp
-L led-driver-rescue:L_Small L1
+L Device:L_Small L1
 U 1 1 59AE9B0A
 P 6050 3850
@@
 $EndComp
 $Comp
-L led-driver-rescue:C_Small C3
+L Device:C_Small C3
 U 1 1 59AE9DC4
 P 5650 2900
@@
 $EndComp
 $Comp
-L led-driver-rescue:C_Small C1
+L Device:C_Small C1
 U 1 1 59AE9F39
 P 2550 3100
@@
 $EndComp
 $Comp
-L led-driver-rescue:GND #PWR01
+L power:GND #PWR01
 U 1 1 59AEA1C1
 P 5800 4100
@@
 $EndComp
 $Comp
-L led-driver-rescue:CONN_01X02 J4
+L Connector_Generic:Conn_01x02 J4
 U 1 1 59AEA206
-P 6950 3900
-F 0 "J4" H 7100 3950 50  0000 C CNN
-F 1 "LED" H 7100 3850 50  0000 C CNN
-F 2 "Pin_Headers:Pin_Header_Straight_1x02_Pitch2.54mm" H 6950 3900 50  0001 C CNN
-F 3 "" H 6950 3900 50  0001 C CNN
-	1    6950 3900
-	1    0    0    -1
-$EndComp
-$Comp
-L led-driver-rescue:GND #PWR02
+P 6950 3850
+F 0 "J4" H 7100 3900 50  0000 C CNN
+F 1 "LED" H 7100 3800 50  0000 C CNN
+F 2 "Pin_Headers:Pin_Header_Straight_1x02_Pitch2.54mm" H 6950 3850 50  0001 C CNN
+F 3 "" H 6950 3850 50  0001 C CNN
+	1    6950 3850
+	1    0    0    -1
+$EndComp
+$Comp
+L power:GND #PWR02
 U 1 1 59AEA35C
 P 6750 4100
@@
 $EndComp
 $Comp
-L led-driver-rescue:GND #PWR03
+L power:GND #PWR03
 U 1 1 59AEA3BF
 P 4350 3750
@@
 $EndComp
 $Comp
-L led-driver-rescue:C_Small C2
+L Device:C_Small C2
 U 1 1 59AEA43B
 P 4250 4100
@@
 $EndComp
 $Comp
-L led-driver-rescue:R_Small R1
+L Device:R_Small R1
 U 1 1 59AEA5E2
 P 4550 4000
@@
 $EndComp
 $Comp
-L led-driver-rescue:GND #PWR04
+L power:GND #PWR04
 U 1 1 59AEA82C
 P 4250 4200
@@
 $EndComp
 $Comp
-L led-driver-rescue:GND #PWR05
+L power:GND #PWR05
 U 1 1 59AEABBE
 P 2550 3200
@@
 $EndComp
 $Comp
-L led-driver-rescue:R_Small R3
+L Device:R_Small R3
 U 1 1 59AEAE7C
 P 4100 2500
@@
 $EndComp
 $Comp
-L led-driver-rescue:R_Small R2
+L Device:R_Small R2
 U 1 1 59AEAEBF
 P 4100 2700
@@
 $EndComp
 $Comp
-L led-driver-rescue:VCC #PWR06
+L power:VCC #PWR06
 U 1 1 59AEAF69
 P 4100 2400
@@
 $EndComp
 $Comp
-L led-driver-rescue:VCC #PWR07
+L power:VCC #PWR07
 U 1 1 59AEAFA4
 P 5800 3200
@@
 $EndComp
 $Comp
-L led-driver-rescue:VCC #PWR08
+L power:VCC #PWR08
 U 1 1 59AEB027
 P 5650 2800
@@
 $EndComp
 $Comp
-L led-driver-rescue:VCC #PWR09
+L power:VCC #PWR09
 U 1 1 59AEB4E1
 P 2550 3000
@@
 $EndComp
 $Comp
-L led-driver-rescue:GND #PWR010
+L power:GND #PWR010
 U 1 1 59AEB7E3
 P 4100 2800
@@
 $EndComp
 $Comp
-L led-driver-rescue:VCC #PWR011
+L power:VCC #PWR011
 U 1 1 59AEBCD0
 P 3700 3500
@@
 $EndComp
 $Comp
-L led-driver-rescue:GND #PWR012
+L power:GND #PWR012
 U 1 1 59AEC65E
 P 3500 3100
@@
 $EndComp
 $Comp
-L led-driver-rescue:CONN_01X02 J3
+L Connector_Generic:Conn_01x02 J3
 U 1 1 59AEC9E5
-P 3300 3050
-F 0 "J3" H 3450 3100 50  0000 C CNN
-F 1 "ADJ" H 3450 3000 50  0000 C CNN
-F 2 "Pin_Headers:Pin_Header_Straight_1x02_Pitch2.54mm" H 3300 3050 50  0001 C CNN
-F 3 "" H 3300 3050 50  0001 C CNN
-	1    3300 3050
+P 3300 3000
+F 0 "J3" H 3450 3050 50  0000 C CNN
+F 1 "ADJ" H 3450 2950 50  0000 C CNN
+F 2 "Pin_Headers:Pin_Header_Straight_1x02_Pitch2.54mm" H 3300 3000 50  0001 C CNN
+F 3 "" H 3300 3000 50  0001 C CNN
+	1    3300 3000
 	-1   0    0    -1
 $EndComp
 $Comp
-L led-driver-rescue:CONN_01X03 J2
+L Connector_Generic:Conn_01x03 J2
 U 1 1 59AED2EC
 P 3500 3600
@@
 $EndComp
 $Comp
-L led-driver-rescue:GND #PWR013
+L power:GND #PWR013
 U 1 1 59AED340
 P 3700 3700
@@
 $EndComp
 $Comp
-L led-driver-rescue:LM3409-RESCUE-led-driver-new U1
+L led-driver:LM3409 U1
 U 1 1 59AEF993
 P 4900 3200
@@
 	3500 3000 3900 3000
 $Comp
-L led-driver-rescue:C_Small C4
+L Device:C_Small C4
 U 1 1 59AF72EA
 P 3900 3100
@@
 $EndComp
 $Comp
-L led-driver-rescue:GND #PWR014
+L power:GND #PWR014
 U 1 1 59AF7850
 P 3900 3200
@@
 Connection ~ 3900 3000
 $Comp
-L led-driver-rescue:C_Small C5
+L Device:C_Small C5
 U 1 1 59AFE85B
 P 6400 3950
@@
 $EndComp
 $Comp
-L led-driver-rescue:GND #PWR015
+L power:GND #PWR015
 U 1 1 59AFEC38
 P 6400 4050
@@
 	4650 4300 6250 4300
 $Comp
-L led-driver-rescue:GND #PWR016
+L power:GND #PWR016
 U 1 1 59B109B8
 P 4900 3900
@@
 $EndComp
 $Comp
-L led-driver-rescue:R_Small R5
+L Device:R_Small R5
 U 1 1 59B11505
 P 6200 3300
@@
 Connection ~ 5800 3400
 $Comp
-L led-driver-rescue:Q_PMOS_GDS Q1
+L Device:Q_PMOS_GDS Q1
 U 1 1 59B006E4
 P 5700 3600
@@
 	5800 3400 6200 3400
 $Comp
-L led-driver-rescue:CONN_01X02 J1
+L Connector_Generic:Conn_01x02 J1
 U 1 1 59AEAC70
-P 1900 3050
-F 0 "J1" H 2050 3100 50  0000 C CNN
-F 1 "48VDC IN" H 2150 3000 50  0000 C CNN
-F 2 "Pin_Headers:Pin_Header_Straight_1x02_Pitch2.54mm" H 1900 3050 50  0001 C CNN
-F 3 "" H 1900 3050 50  0001 C CNN
-	1    1900 3050
+P 1900 3000
+F 0 "J1" H 2050 3050 50  0000 C CNN
+F 1 "48VDC IN" H 2150 2950 50  0000 C CNN
+F 2 "Pin_Headers:Pin_Header_Straight_1x02_Pitch2.54mm" H 1900 3000 50  0001 C CNN
+F 3 "" H 1900 3000 50  0001 C CNN
+	1    1900 3000
 	-1   0    0    -1
 $EndComp
